File: kicad/pico-radio-5/pico-radio-5.kicad_sch (KiCad schematic)
At the start: 45 parts, among them J1 HF Amplifier, J2 MW/SW antenna, J3 FM antenna, J4 SW antenna, J5 Batterry, Q1 PN2222A, Q2 PN2222A, Q3 PN2222A, SW1 Reset, U1 SI4732-A10-GS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

Commit message: Refactor code structure for improved readability and maintainability
Parts:
- C3: value 100nF -> 22nF
- R3, R4: value 22k -> 1k
Changed lines of the file:
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@@
 			)
 		)
-		(property "Value" "22k"
+		(property "Value" "1k"
 			(at 184.15 133.35 90)
 			(effects
@@
 			)
 		)
-		(property "Value" "100nF"
+		(property "Value" "22nF"
 			(at 196.85 137.16 90)
 			(effects
@@
 			)
 		)
-		(property "Value" "22k"
+		(property "Value" "1k"
 			(at 184.15 143.51 90)
 			(effects
