File: kicad/pico-radio-9-kétoldalas/pico-radio-9-kétoldalas.kicad_pcb (KiCad board)
At the start: 2 copper layers, 54 parts, among them J1 FM antenna, J2 SW antenna, J3 MW/SW antenna kapcsoló, J4 HF Amplifier, J5 Batterry, Q1 PN2222A, Q2 PN2222A, Q3 PN2222A, SW1 Reset, U1 SI4732-A10-GS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

Commit message: Dual side PCB
Parts:
- removed H4: MountingHole, MountingHole:MountingHole_3.2mm_M3
- removed JP2: Si4732 I2C Address, Jumper:SolderJumper-3_P1.3mm_Bridged12_RoundedPad1.0x1.5mm
- moved R12 220.5 mm to (130.5, 47.8), turned to -90 degrees
- moved R13 215.4 mm to (125.8, 58.0), turned to -90 degrees
- moved C12 180.5 mm to (125.0, 35.2), turned to -90 degrees
- moved C11 177.0 mm to (130.0, 35.2), turned to -90 degrees
- moved H1 174.7 mm to (136.8, 83.8)
- moved H2 174.3 mm to (136.8, 33.5)
- moved L1 166.9 mm to (63.1, 75.2)
- moved L3 164.1 mm to (63.2, 71.7)
- moved R4 164.0 mm to (71.2, 64.8), turned to 90 degrees
- moved J5 163.0 mm to (135.2, 43.0), turned to -90 degrees
- moved R3 161.7 mm to (68.0, 64.7), turned to 90 degrees
- moved R2 158.2 mm to (64.5, 60.3), turned to 90 degrees
- moved R1 155.8 mm to (61.0, 60.2), turned to 90 degrees
- moved SW1 152.3 mm to (125.0, 48.0)
- moved C10 140.7 mm to (88.5, 60.2), turned to 90 degrees
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Connections:
- J4 pad 2: AUDIO_R -> AUDIO_L
- J4 pad 3: AUDIO_L -> AUDIO_R
- RV1 pad 1: AD_FFT_AUDIO -> Net-(R11-Pad1)
- RV1 pad 3: Net-(R11-Pad1) -> AD_FFT_AUDIO
- U1 pad 10: Net-(JP2-C) -> GND
Routing:
- net GND: track 107.2 -> 407.8 mm
- net +3.3V: track 15.6 -> 144.0 mm
- net AD_FFT_AUDIO: track 0.00 -> 90.0 mm
- net +Vbus: track 0.00 -> 89.0 mm
- net AUDIO_MUTE: track 0.00 -> 85.7 mm
- net AUDIO_L: track 0.00 -> 60.7 mm
- net AUDIO_R: track 0.00 -> 59.1 mm
- net Net-(U3B-+): track 0.00 -> 38.9 mm
- net Net-(U3B--): track 0.00 -> 24.1 mm
- net Net-(JP2-C): track 21.5 -> 0.00 mm
- net Net-(J3-Pin_2): track 0.00 -> 17.0 mm
- net Net-(J3-Pin_3): track 0.00 -> 15.9 mm
- net Net-(Q2-B): track 0.00 -> 14.2 mm
- net Net-(J1-Pin_2): track 0.00 -> 13.8 mm
- net Net-(C7-Pad1): track 0.00 -> 11.7 mm
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Other:
- board outline added: 88 x 57.2 mm
- board text added: "Pico Radio V9 BT-Soft 2025"
