File: kicad/pico-radio-9-kétoldalas/pico-radio-9-kétoldalas.kicad_pcb (KiCad board)
At the start: 2 copper layers, 88 x 57.2 mm, 52 parts, among them J1 FM antenna, J2 SW antenna, J3 MW/SW antenna kapcsoló, J4 HF Amplifier, J5 Batterry, Q1 PN2222A, Q2 PN2222A, Q3 PN2222A, SW1 Reset, U1 SI4732-A10-GS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

Commit message: Dual sided  PCB update
Parts:
- removed U4: KY-040, Rotary_Encoder:KY-040-PORT
- added H4: MountingHole, MountingHole:MountingHole_3.2mm_M3, F.Cu at (89.8, 50.0)
- added J6: KY-040 Rotary, Connector_PinHeader_2.54mm:PinHeader_1x05_P2.54mm_Vertical, F.Cu at (94.8, 83.4)
Routing:
- net GND: track 407.8 -> 409.0 mm
